File: hardware/musicboard.sch (KiCad schematic (older format))
At the start: 74 parts, among them J1 USB_B_Micro, J2 AudioJack3, J3 AudioJack3, J4 AudioJack3, J5 Conn_01x02_Female, J6 Conn_01x02_Female, J7 Conn_01x04_Female, J8 Conn_01x06_Female, SW1 SW_Push, U1 STM32F745VETx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

Commit message: add extension to board + add former fluidsynth
Parts:
- added D2: LED, LED_SMD:LED_0603_1608Metric_Pad1.05x0.95mm_HandSolder, symbol Device:LED
- added J9: Conn_01x03_Female, Connector_PinHeader_2.54mm:PinHeader_1x03_P2.54mm_Vertical, symbol Connector:Conn_01x04_Female
- added R19: 1k, Resistor_SMD:R_0603_1608Metric_Pad1.05x0.95mm_HandSolder, symbol Device:R
- J7: footprint Connector_PinHeader_2.54mm:PinHeader_1x04_P2.54mm_Vertical -> Connector_PinHeader_2.54mm:PinHeader_1x08_P2.54mm_Vertical; symbol Connector:Conn_01x04_Female -> Connector:Conn_01x08_Female
Connections:
- net GND: now also J7.8 (Pin_8), D2.1 (K); no longer J7.4 (Pin_4)
- net GNDA: now also J9.4 (Pin_4)
- net VDDA: now also J9.1 (Pin_1)
- net EXT_SCL: now reaches U1.46 (PB10)
- net EXT_SCL: now also J7.2 (Pin_2)
- net EXT_SDA: now reaches U1.47 (PB11)
- net EXT_SDA: now also J7.3 (Pin_3)
- net TX2: now reaches U1.78 (PC10)
- net TX2: now also J7.4 (Pin_4)
- net RX2: now reaches U1.79 (PC11)
- net RX2: now also J7.5 (Pin_5)
- net LED2: now reaches U1.80 (PC12)
- net LED2: now also R19.2
- net MICBIAS: now reaches U4.17 (MICBIAS)
- net MICBIAS: now also J9.3 (Pin_3)
- net MICIN: now reaches U4.18 (MICIN)
- net MICIN: now also J9.2 (Pin_2)
- net LED renamed LED1
- net RX renamed RX1
- net RX1: now also J7.7 (Pin_7); no longer J7.3 (Pin_3)
- net TX renamed TX1
- net TX1: now also J7.6 (Pin_6); no longer J7.2 (Pin_2)
- new net: D2.2 (A), R19.1
Other:
- moved on the sheet: C10, C11, C12, C13, C15, C16, C17, C18, C6, C7, C8, D1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

Commit message: use usb mini b + add usb header
Parts:
- removed J1: USB_B_Micro, Connector_USB:USB_Micro-B_Molex-105017-0001, symbol Connector:USB_B_Micro
- added J1: USB_B_Mini, hardware:USB-mini-B-0548190519, symbol Connector:USB_B_Mini
- added J?: Conn_01x02_Female, Connector_PinHeader_2.54mm:PinHeader_1x02_P2.54mm_Vertical, symbol Connector:Conn_01x02_Female
- J9: value Conn_01x03_Female -> Conn_01x04_Female; footprint Connector_PinHeader_2.54mm:PinHeader_1x03_P2.54mm_Vertical -> Connector_PinHeader_2.54mm:PinHeader_1x04_P2.54mm_Vertical
Connections:
- net +5V: now also J1.1 (VBUS)
- net GND: now also J1.5 (GND), J1.6 (Shield)
- net DM: now reaches R4.2
- net DM: now also J1.2 (D-), J?.2 (Pin_2)
- net DP: now reaches R3.2
- net DP: now also J1.3 (D+), J?.1 (Pin_1)
Other:
- moved on the sheet: J5, J7
Changed lines of the file:
@@
-	1    0    0    -1
-$EndComp
-$Comp
-L Connector:USB_B_Micro J1
-U 1 1 5ED878CD
-P 5050 3650
-F 0 "J1" H 5107 4117 50  0000 C CNN
-F 1 "USB_B_Micro" H 5107 4026 50  0000 C CNN
-F 2 "Connector_USB:USB_Micro-B_Molex-105017-0001" H 5200 3600 50  0001 C CNN
-F 3 "~" H 5200 3600 50  0001 C CNN
-	1    5050 3650
 	1    0    0    -1
 $EndComp
@@
 L Connector:Conn_01x02_Female J5
 U 1 1 5F05FF1E
-P 5100 4950
-F 0 "J5" H 5128 4926 50  0000 L CNN
-F 1 "Conn_01x02_Female" H 5128 4835 50  0000 L CNN
-F 2 "Connector_PinHeader_2.54mm:PinHeader_1x02_P2.54mm_Vertical" H 5100 4950 50  0001 C CNN
-F 3 "~" H 5100 4950 50  0001 C CNN
-	1    5100 4950
-	1    0    0    -1
-$EndComp
-Wire Wire Line
-	4900 5050 4700 5050
-Wire Wire Line
-	4900 4950 4700 4950
-Text Label 4700 5050 0    50   ~ 0
+P 5150 5300
+F 0 "J5" H 5178 5276 50  0000 L CNN
+F 1 "Conn_01x02_Female" H 5178 5185 50  0000 L CNN
+F 2 "Connector_PinHeader_2.54mm:PinHeader_1x02_P2.54mm_Vertical" H 5150 5300 50  0001 C CNN
+F 3 "~" H 5150 5300 50  0001 C CNN
+	1    5150 5300
+	1    0    0    -1
+$EndComp
+Wire Wire Line
+	4950 5400 4750 5400
+Wire Wire Line
+	4950 5300 4750 5300
+Text Label 4750 5400 0    50   ~ 0
 BOOT0
-Text Label 4700 4950 0    50   ~ 0
+Text Label 4750 5300 0    50   ~ 0
 VDD
 $Comp
 L Connector:Conn_01x08_Female J7
 U 1 1 5F0B3786
-P 5100 5600
-F 0 "J7" H 5128 5576 50  0000 L CNN
-F 1 "Conn_01x04_Female" H 5128 5485 50  0000 L CNN
-F 2 "Connector_PinHeader_2.54mm:PinHeader_1x08_P2.54mm_Vertical" H 5100 5600 50  0001 C CNN
-F 3 "~" H 5100 5600 50  0001 C CNN
-	1    5100 5600
-	1    0    0    -1
-$EndComp
-Wire Wire Line
-	4900 5300 4600 5300
-Wire Wire Line
-	4900 5700 4600 5700
-Wire Wire Line
-	4900 5600 4600 5600
-Wire Wire Line
-	4900 6000 4600 6000
-Text Label 4600 6000 0    50   ~ 0
+P 5150 5950
+F 0 "J7" H 5178 5926 50  0000 L CNN
+F 1 "Conn_01x04_Female" H 5178 5835 50  0000 L CNN
+F 2 "Connector_PinHeader_2.54mm:PinHeader_1x08_P2.54mm_Vertical" H 5150 5950 50  0001 C CNN
+F 3 "~" H 5150 5950 50  0001 C CNN
+	1    5150 5950
+	1    0    0    -1
+$EndComp
+Wire Wire Line
+	4950 5650 4650 5650
+Wire Wire Line
+	4950 6050 4650 6050
+Wire Wire Line
+	4950 5950 4650 5950
+Wire Wire Line
+	4950 6350 4650 6350
+Text Label 4650 6350 0    50   ~ 0
 GND
-Text Label 4600 5300 0    50   ~ 0
+Text Label 4650 5650 0    50   ~ 0
 VDD
-Text Label 4600 5600 0    50   ~ 0
+Text Label 4650 5950 0    50   ~ 0
 TX2
-Text Label 4600 5700 0    50   ~ 0
+Text Label 4650 6050 0    50   ~ 0
 RX2
 $Comp
@@
 EXT_SDA
 Wire Wire Line
-	4900 5400 4600 5400
-Wire Wire Line
-	4900 5500 4600 5500
-Text Label 4600 5400 0    50   ~ 0
+	4950 5750 4650 5750
+Wire Wire Line
+	4950 5850 4650 5850
+Text Label 4650 5750 0    50   ~ 0
 EXT_SCL
-Text Label 4600 5500 0    50   ~ 0
+Text Label 4650 5850 0    50   ~ 0
 EXT_SDA
 Wire Wire Line
@@
 RX2
 Wire Wire Line
-	4900 5900 4600 5900
-Wire Wire Line
-	4900 5800 4600 5800
-Text Label 4600 5800 0    50   ~ 0
+	4950 6250 4650 6250
+Wire Wire Line
+	4950 6150 4650 6150
+Text Label 4650 6150 0    50   ~ 0
 TX1
-Text Label 4600 5900 0    50   ~ 0
+Text Label 4650 6250 0    50   ~ 0
 RX1
 Wire Wire Line
@@
 P 7450 3800
 F 0 "J9" H 7478 3776 50  0000 L CNN
-F 1 "Conn_01x03_Female" H 7478 3685 50  0000 L CNN
-F 2 "Connector_PinHeader_2.54mm:PinHeader_1x03_P2.54mm_Vertical" H 7450 3800 50  0001 C CNN
+F 1 "Conn_01x04_Female" H 7478 3685 50  0000 L CNN
+F 2 "Connector_PinHeader_2.54mm:PinHeader_1x04_P2.54mm_Vertical" H 7450 3800 50  0001 C CNN
 F 3 "~" H 7450 3800 50  0001 C CNN
 	1    7450 3800
@@
 Text Label 6950 3700 0    50   ~ 0
 VDDA
+$Comp
+L Connector:USB_B_Mini J1
+U 1 1 5EEAA8F5
+P 5050 3650
+F 0 "J1" H 5107 4117 50  0000 C CNN
+F 1 "USB_B_Mini" H 5107 4026 50  0000 C CNN
+F 2 "hardware:USB-mini-B-0548190519" H 5200 3600 50  0001 C CNN
+F 3 "~" H 5200 3600 50  0001 C CNN
+	1    5050 3650
+	1    0    0    -1
+$EndComp
+$Comp
+L Connector:Conn_01x02_Female J?
+U 1 1 5EEB19CC
+P 5100 4850
+F 0 "J?" H 5128 4826 50  0000 L CNN
+F 1 "Conn_01x02_Female" H 5128 4735 50  0000 L CNN
+F 2 "Connector_PinHeader_2.54mm:PinHeader_1x02_P2.54mm_Vertical" H 5100 4850 50  0001 C CNN
+F 3 "~" H 5100 4850 50  0001 C CNN
+	1    5100 4850
+	1    0    0    -1
+$EndComp
+Wire Wire Line
+	4900 4850 4700 4850
+Wire Wire Line
+	4900 4950 4700 4950
+Text Label 5500 3650 0    50   ~ 0
+DP
+Text Label 5500 3750 0    50   ~ 0
+DM
+Text Label 4700 4850 0    50   ~ 0
+DP
+Text Label 4700 4950 0    50   ~ 0
+DM
 $EndSCHEMATC

Commit message: update schematics
Parts:
- gave numbers to parts that had none: 1
Changed lines of the file:
@@
 $EndComp
 $Comp
-L Connector:Conn_01x02_Female J?
+L Connector:Conn_01x02_Female J10
 U 1 1 5EEB19CC
 P 5100 4850
-F 0 "J?" H 5128 4826 50  0000 L CNN
+F 0 "J10" H 5128 4826 50  0000 L CNN
 F 1 "Conn_01x02_Female" H 5128 4735 50  0000 L CNN
 F 2 "Connector_PinHeader_2.54mm:PinHeader_1x02_P2.54mm_Vertical" H 5100 4850 50  0001 C CNN

Commit message: misc
Parts:
- J2, J3, J4: Alt (none) -> http://www.switchcraft.com/Drawings/35rapc__v4_cd.pdf
- U2: Alt (none) -> http://ww1.microchip.com/downloads/en/DeviceDoc/21373C.pdf
Changed lines of the file:
@@
 F 1 "AudioJack3" H 10220 5784 50  0000 R CNN
 F 2 "Connector_Audio:Jack_3.5mm_CUI_SJ1-3535NG_Horizontal" H 10500 5850 50  0001 C CNN
-F 3 "~" H 10500 5850 50  0001 C CNN
+F 3 "https://www.cuidevices.com/product/resource/sj1-353xng.pdf" H 10500 5850 50  0001 C CNN
+F 4 "http://www.switchcraft.com/Drawings/35rapc__v4_cd.pdf" H 10500 5850 50  0001 C CNN "Alt"
 	1    10500 5850
 	-1   0    0    -1
@@
 F 1 "AudioJack3" H 10220 5334 50  0000 R CNN
 F 2 "Connector_Audio:Jack_3.5mm_CUI_SJ1-3535NG_Horizontal" H 10500 5400 50  0001 C CNN
-F 3 "~" H 10500 5400 50  0001 C CNN
+F 3 "https://www.cuidevices.com/product/resource/sj1-353xng.pdf" H 10500 5400 50  0001 C CNN
+F 4 "http://www.switchcraft.com/Drawings/35rapc__v4_cd.pdf" H 10500 5400 50  0001 C CNN "Alt"
 	1    10500 5400
 	-1   0    0    -1
@@
 F 1 "AudioJack3" H 10220 4834 50  0000 R CNN
 F 2 "Connector_Audio:Jack_3.5mm_CUI_SJ1-3535NG_Horizontal" H 10500 4900 50  0001 C CNN
-F 3 "~" H 10500 4900 50  0001 C CNN
+F 3 "https://www.cuidevices.com/product/resource/sj1-353xng.pdf" H 10500 4900 50  0001 C CNN
+F 4 "http://www.switchcraft.com/Drawings/35rapc__v4_cd.pdf" H 10500 4900 50  0001 C CNN "Alt"
 	1    10500 4900
 	-1   0    0    -1
@@
 F 2 "Package_TO_SOT_SMD:SOT-223-3_TabPin2" H 5450 7200 50  0001 C CNN
 F 3 "http://ww1.microchip.com/downloads/en/devicedoc/22056b.pdf" H 5550 7300 50  0001 C CNN
+F 4 "http://ww1.microchip.com/downloads/en/DeviceDoc/21373C.pdf" H 5550 7050 50  0001 C CNN "Alt"
 	1    5550 7050
 	1    0    0    -1
